File: schematics/v2_ordered/Humus_ethernet_dip_v2.brd (EAGLE design)
At the start: 41 x 50 mm, 31 parts

Commit message: moved folder to v2_ordered
Parts:
- removed PAD1: (no value), wirepad:SMD2,54-5,08
- removed R3: (no value), rcl:R0805
- removed U$1: HFJT1, CONNECTER:HFJT1
- added IC2: DS2432P, 1wire:TSOC6
- added R10: (no value), rcl:R0805
- PAD3: value (none) -> WIREPADSMD1,27-254; device wirepad:SMD2,54-5,08 -> wirepad:SMD1,27-2,54
- moved U$5 50.6 mm to (6.95, 37.5)
- moved RJ1 38.0 mm to (25.4, 43.6), turned to 90 degrees
- moved C3 29.2 mm to (13.3, 3.50), flipped to the top
- moved R9 23.5 mm to (29.4, 22.1), flipped to the top
- moved R8 23.0 mm to (24.1, 22.1), flipped to the top
- moved C4 21.8 mm to (14.2, 9.50), flipped to the top
- moved C1 21.5 mm to (32.4, 5.30), flipped to the top, turned to 0 degrees
- moved C5 19.4 mm to (14.2, 7.40), flipped to the top, turned to 0 degrees
- moved FB1 19.3 mm to (32.7, 29.1), flipped to the top, turned to 180 degrees
- moved C7 19.3 mm to (14.2, 14.8), flipped to the top, turned to 0 degrees
- moved C10 19.0 mm to (32.7, 31.2), flipped to the top
- moved R2 17.9 mm to (33.0, 16.1), flipped to the top, turned to 0 degrees
- moved Q1 16.4 mm to (8.90, 11.6), flipped to the top, turned to 270 degrees
- moved C8 16.2 mm to (14.2, 17.4), flipped to the top, turned to 0 degrees
- moved C6 15.9 mm to (14.2, 12.7), flipped to the top, turned to 0 degrees
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Connections:
- removed net 3V3: SV2.31
- removed net N$12: PAD1.1, U1.4
- removed net NC1: U$1.7
- removed net NC2: U$1.8
- removed net PW+: U$1.9
- removed net PW-: U$1.10
- net AP2: now also U1.4
- net CSIPCK: now also U1.9
- net CT: no longer U$1.3
- net D0: no longer R3.1, U1.9
- net GND: now also IC2.4; no longer U$1.12, U$1.14, U$1.6
- net LD2: now also IC2.3, R10.1
- net N$10: no longer U$1.11
- net N$11: no longer U$1.13
- net RD+: no longer U$1.4
- net RD-: no longer U$1.5
- net TD+: no longer U$1.1
- net TD-: no longer U$1.2
- net VDD: now also R10.2, SV2.31; no longer R3.2
Routing:
- net VDD: track 0.00 -> 187.7 mm
- net GND: track 0.00 -> 66.7 mm, vias 0 -> 10
- net RD+: track 0.00 -> 40.2 mm, vias 0 -> 2
- net TD+: track 0.00 -> 38.8 mm, vias 0 -> 2
- net N$11: track 0.00 -> 32.2 mm, vias 0 -> 1
- net N$10: track 0.00 -> 30.8 mm, vias 0 -> 1
- net RD-: track 0.00 -> 30.7 mm, vias 0 -> 1
- net N$16: track 0.00 -> 27.8 mm, vias 0 -> 2
- net TD-: track 0.00 -> 26.8 mm, vias 0 -> 2
- net N$15: track 0.00 -> 22.0 mm, vias 0 -> 2
- net N$7: track 0.00 -> 21.1 mm
- net N$6: track 0.00 -> 20.9 mm
- net LD2: track 0.00 -> 19.0 mm, vias 0 -> 1
- net AP2: track 0.00 -> 16.0 mm, vias 0 -> 1
- net CSVSYNC: track 0.00 -> 14.7 mm
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- added copper zone on layer 1, net CT
- added copper zone on layer 1, net VDD
- removed copper zone on layer 1, net GND
Other:
- outline, holes or cut-outs redrawn
- board text added: "C.H.I.P. HUMUS DIP"
- board text added: "JKW v0.2"
- board text removed: "JKW v0.43"
- board text removed: "QUESO DIP"
