File: schematics/v3_ordered/Humus_ethernet_dip_v3.brd (EAGLE design)
At the start: 41 x 50 mm, 31 parts, among them IC2 DS2432P

Commit message: fixed ds2431
Parts:
- removed IC2: DS2432P, 1wire:TSOC6
- added U2: DS2431P, JKW_CHIP:TSOC6
Connections:
- net GND: now also U2.1; no longer IC2.4
- net LD2: now also U2.2; no longer IC2.3
Routing:
- net GND: track 64.5 -> 64.6 mm, vias 9 -> 10
Changed lines of the file:
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@@
 <?xml version="1.0" encoding="utf-8"?>
 <!DOCTYPE eagle SYSTEM "eagle.dtd">
-<eagle version="6.5.0">
+<eagle version="7.6.0">
 <drawing>
 <settings>
@@
 <layers>
 <layer number="1" name="Top" color="4" fill="1" visible="yes" active="yes"/>
+<layer number="2" name="Route2" color="1" fill="3" visible="yes" active="yes"/>
+<layer number="3" name="Route3" color="4" fill="3" visible="yes" active="yes"/>
+<layer number="14" name="Route14" color="1" fill="6" visible="yes" active="yes"/>
+<layer number="15" name="Route15" color="4" fill="6" visible="yes" active="yes"/>
 <layer number="16" name="Bottom" color="1" fill="1" visible="yes" active="yes"/>
 <layer number="17" name="Pads" color="2" fill="1" visible="yes" active="yes"/>
@@
 <layer number="56" name="wert" color="7" fill="1" visible="no" active="no"/>
 <layer number="57" name="tCAD" color="7" fill="1" visible="no" active="no"/>
-<layer number="90" name="Modules" color="5" fill="1" visible="no" active="yes"/>
+<layer number="59" name="tCarbon" color="7" fill="1" visible="yes" active="yes"/>
+<layer number="60" name="bCarbon" color="7" fill="1" visible="yes" active="yes"/>
+<layer number="90" name="Modules" color="5" fill="1" visible="no" active="no"/>
 <layer number="91" name="Nets" color="2" fill="1" visible="no" active="no"/>
 <layer number="92" name="Busses" color="1" fill="1" visible="no" active="no"/>
@@
 <layer number="113" name="IDFDebug" color="7" fill="1" visible="no" active="yes"/>
 <layer number="116" name="Patch_BOT" color="9" fill="4" visible="yes" active="yes"/>
+<layer number="118" name="Rect_Pads" color="7" fill="1" visible="yes" active="yes"/>
 <layer number="121" name="_tsilk" color="7" fill="1" visible="yes" active="yes"/>
 <layer number="122" name="_bsilk" color="7" fill="1" visible="yes" active="yes"/>
@@
 <layer number="127" name="_tValues" color="7" fill="1" visible="no" active="yes"/>
 <layer number="128" name="_bValues" color="7" fill="1" visible="no" active="yes"/>
+<layer number="129" name="Mask" color="7" fill="1" visible="yes" active="yes"/>
 <layer number="131" name="tAdjust" color="7" fill="1" visible="no" active="yes"/>
 <layer number="132" name="bAdjust" color="7" fill="1" visible="no" active="yes"/>
@@
 <layer number="154" name="FabDoc2" color="7" fill="1" visible="no" active="yes"/>
 <layer number="155" name="FabDoc3" color="7" fill="1" visible="no" active="yes"/>
+<layer number="156" name="tAssmbl" color="7" fill="1" visible="yes" active="yes"/>
+<layer number="157" name="bAssmbl" color="7" fill="1" visible="yes" active="yes"/>
 <layer number="199" name="Contour" color="7" fill="1" visible="no" active="yes"/>
 <layer number="200" name="200bmp" color="1" fill="10" visible="no" active="yes"/>
@@
 <layer number="223" name="223bmp" color="24" fill="1" visible="no" active="no"/>
 <layer number="224" name="224bmp" color="25" fill="1" visible="no" active="no"/>
+<layer number="225" name="225bmp" color="7" fill="1" visible="yes" active="yes"/>
+<layer number="226" name="226bmp" color="7" fill="1" visible="yes" active="yes"/>
+<layer number="227" name="227bmp" color="7" fill="1" visible="yes" active="yes"/>
+<layer number="228" name="228bmp" color="7" fill="1" visible="yes" active="yes"/>
+<layer number="229" name="229bmp" color="7" fill="1" visible="yes" active="yes"/>
+<layer number="230" name="230bmp" color="7" fill="1" visible="yes" active="yes"/>
+<layer number="231" name="Eagle3D_PG1" color="7" fill="1" visible="yes" active="yes"/>
+<layer number="232" name="Eagle3D_PG2" color="7" fill="1" visible="yes" active="yes"/>
+<layer number="233" name="Eagle3D_PG3" color="7" fill="1" visible="yes" active="yes"/>
 <layer number="248" name="Housing" color="7" fill="1" visible="no" active="yes"/>
 <layer number="249" name="Edge" color="7" fill="1" visible="no" active="yes"/>
@@
 <layer number="251" name="SMDround" color="12" fill="11" visible="no" active="no"/>
 <layer number="254" name="cooling" color="7" fill="1" visible="yes" active="yes"/>
+<layer number="255" name="logo" color="7" fill="1" visible="yes" active="yes"/>
 </layers>
 <board>
@@
 <pass name="Default">
 <param name="RoutingGrid" value="50mil"/>
+<param name="AutoGrid" value="1"/>
+<param name="Efforts" value="0"/>
+<param name="TopRouterVariant" value="1"/>
 <param name="tpViaShape" value="round"/>
 <param name="PrefDir.1" value="|"/>
@@
 <attribute name="VALUE" x="24.435" y="25.84" size="1.27" layer="27" rot="R180"/>
 </element>
-<element name="IC2" library="1wire" package="TSOC6" value="DS2432P" x="16.45" y="46.3" smashed="yes" rot="R180"/>
 <element name="R10" library="rcl" package="R0805" value="" x="12.25" y="46.3" smashed="yes" rot="R270">
 <attribute name="VALUE" x="9.71" y="46.935" size="1.27" layer="27" rot="R270"/>
@@
 <element name="USB" library="Spark" package="USB-MICROB-SMT-DIP" value="USBUSB-MICROB-SMT-DIP" x="26.7" y="48.55" smashed="yes" rot="R180">
 <attribute name="NAME" x="28.3" y="49" size="0.762" layer="25" rot="R180"/>
+</element>
+<element name="U2" library="JKW_CHIP" package="TSOC6" value="DS2431P" x="15.6" y="46.1" smashed="yes" rot="R180">
+<attribute name="TOLLERANCE" value="" x="15.6" y="46.1" size="1.778" layer="27" rot="R180" display="off"/>
+<attribute name="MFG_PN" value="DS2431P+T&amp;RCT-ND" x="15.6" y="46.1" size="1.778" layer="27" rot="R180" display="off"/>
+<attribute name="DESCRIPTION" value="IC, 1024-Bit, 1-Wire EEPROM, TSOC6" x="15.6" y="46.1" size="1.778" layer="27" rot="R180" display="off"/>
+<attribute name="ASSEMBLE" value="" x="15.6" y="46.1" size="1.778" layer="27" rot="R180" display="off"/>
+<attribute name="VENDOR" value="MAXIM" x="15.6" y="46.1" size="1.778" layer="27" rot="R180" display="off"/>
+<attribute name="VENDOR_PART_NUMBER" value="DS2431P+T&amp;R" x="15.6" y="46.1" size="1.778" layer="27" rot="R180" display="off"/>
+<attribute name="MFG" value="DIGIKEY" x="15.6" y="46.1" size="1.778" layer="27" rot="R180" display="off"/>
+<attribute name="PART_TYPE" value="IC" x="15.6" y="46.1" size="1.778" layer="27" rot="R180" display="off"/>
+<attribute name="PRICE" value="0.98" x="15.6" y="46.1" size="1.778" layer="27" rot="R180" display="off"/>
+<attribute name="LINK" value="http://www.digikey.com/product-detail/en/DS2431P%2BT%26R/DS2431P%2BT%26RCT-ND/3647900" x="15.6" y="46.1" size="1.778" layer="27" rot="R180" display="off"/>
+<attribute name="FOOTPRINT" value="TSOC6" x="15.6" y="46.1" size="1.778" layer="27" rot="R180" display="off"/>
+<attribute name="NAME" x="16.94" y="46.76" size="1.27" layer="25" font="vector" rot="R180"/>
+<attribute name="VALUE" x="17.99" y="47.29" size="1.27" layer="27" font="vector" rot="R270"/>
 </element>
 </elements>
@@
 <wire x1="24.775" y1="30.475" x2="23.95" y2="29.65" width="0.4064" layer="1"/>
 <wire x1="23.95" y1="29.65" x2="23.95" y2="28.25" width="0.4064" layer="1"/>
-<contactref element="IC2" pad="4"/>
-<contactref element="IC2" pad="4"/>
 <via x="17.05" y="37.1" extent="1-16" drill="0.6"/>
 <via x="17.2" y="34.2" extent="1-16" drill="0.6"/>
@@
 <wire x1="17.825" y1="36.325" x2="17.05" y2="37.1" width="0.3048" layer="1"/>
 <wire x1="15.05" y1="42.7" x2="15.18" y2="42.83" width="0.254" layer="1"/>
-<wire x1="15.18" y1="42.83" x2="15.18" y2="44.6998" width="0.254" layer="1"/>
 <via x="33.45" y="42.25" extent="1-16" drill="0.6"/>
 <via x="30.15" y="21.6" extent="1-16" drill="0.6"/>
@@
 <wire x1="16.4" y1="14.95" x2="16.4" y2="17.35" width="0.254" layer="1"/>
 <wire x1="16.4" y1="17.35" x2="14.7" y2="19.05" width="0.254" layer="1"/>
+<contactref element="U2" pad="1"/>
+<via x="18.75" y="47.9" extent="1-16" drill="0.6"/>
+<wire x1="16.87" y1="47.7002" x2="18.5502" y2="47.7002" width="0.254" layer="1"/>
+<wire x1="18.5502" y1="47.7002" x2="18.75" y2="47.9" width="0.254" layer="1"/>
 </signal>
 <signal name="INT0">
@@
 <signal name="LD2">
 <contactref element="SV2" pad="19"/>
-<contactref element="IC2" pad="3"/>
 <contactref element="R10" pad="1"/>
 <wire x1="1.45" y1="24.27" x2="2.7" y2="25.52" width="0.254" layer="1"/>
@@
 <wire x1="2.7" y1="43.15" x2="3.05" y2="43.5" width="0.254" layer="1"/>
 <wire x1="12.45" y1="48.85" x2="15.05" y2="48.85" width="0.254" layer="1"/>
-<wire x1="15.05" y1="48.85" x2="15.2" y2="48.7" width="0.254" layer="1"/>
-<wire x1="15.2" y1="48.7" x2="15.2" y2="47.9202" width="0.254" layer="1"/>
-<wire x1="15.2" y1="47.9202" x2="15.18" y2="47.9002" width="0.254" layer="1"/>
 <wire x1="12.25" y1="47.25" x2="12.25" y2="48.65" width="0.254" layer="1"/>
 <wire x1="12.25" y1="48.65" x2="12.45" y2="48.85" width="0.254" layer="1"/>
@@
 <wire x1="6.55" y1="44.65" x2="5.4" y2="43.5" width="0.254" layer="1"/>
 <wire x1="5.4" y1="43.5" x2="3.05" y2="43.5" width="0.254" layer="1"/>
+<contactref element="U2" pad="2"/>
+<wire x1="15.6" y1="47.7002" x2="15.6" y2="48.3" width="0.254" layer="1"/>
+<wire x1="15.6" y1="48.3" x2="15.05" y2="48.85" width="0.254" layer="1"/>
 </signal>
 <signal name="LD4">
