File: schematics/v4_ordered/Humus_ethernet_dip_v4.brd (EAGLE design)
At the start: 41 x 50 mm, 31 parts, among them Q1 25MHz, U1 ENC28J60SS, U2 DS2431P

Commit message: updated
Parts:
- removed U$5: LOGO_10X10_SILK, logo:LOGO_10X10_SILK
- added U$1: LOGO_10X10_SILK, JKW_CHIP:LOGO2_10X10_SILK
