File: schematics/v4_ordered/Humus_ethernet_dip_v4.sch (EAGLE design)
At the start: 31 parts, among them Q1 25MHz, U1 ENC28J60SS, U2 DS2431P

Commit message: updated
Parts:
- removed U$5: LOGO_10X10_SILK, logo:LOGO_10X10_SILK
- added U$1: LOGO_10X10_SILK, JKW_CHIP:LOGO_10X10_SILK
Changed lines of the file:
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@@
 <layer number="112" name="tSilk" color="7" fill="1" visible="yes" active="yes"/>
 <layer number="113" name="IDFDebug" color="7" fill="1" visible="yes" active="yes"/>
+<layer number="114" name="Badge_Outline" color="7" fill="1" visible="yes" active="yes"/>
+<layer number="115" name="ReferenceISLANDS" color="7" fill="1" visible="yes" active="yes"/>
 <layer number="116" name="Patch_BOT" color="9" fill="4" visible="yes" active="yes"/>
 <layer number="118" name="Rect_Pads" color="7" fill="1" visible="yes" active="yes"/>
@@
 <part name="U$4" library="logo" deviceset="LOGO_3X3_COPPER" device=""/>
 <part name="U$2" library="logo" deviceset="LOGO_3X3_COPPER" device=""/>
-<part name="U$5" library="logo" deviceset="LOGO_10X10_SILK" device=""/>
 <part name="U1" library="SparkFun-DigitalIC" deviceset="ENC28J60" device="" value="ENC28J60SS"/>
 <part name="RJ1" library="CONNECTER" deviceset="HR911105A" device=""/>
@@
 <part name="GND4" library="supply1" deviceset="GND" device=""/>
 <part name="U2" library="JKW_CHIP" deviceset="DS2431" device="P"/>
+<part name="U$1" library="JKW_CHIP" deviceset="LOGO_10X10_SILK" device=""/>
 </parts>
 <sheets>
@@
 <instance part="U$4" gate="G$1" x="91.44" y="2.54"/>
 <instance part="U$2" gate="G$1" x="5.08" y="2.54"/>
-<instance part="U$5" gate="G$1" x="177.8" y="2.54"/>
 <instance part="U1" gate="G$1" x="91.44" y="182.88"/>
 <instance part="RJ1" gate="G$1" x="246.38" y="175.26"/>
@@
 <instance part="GND4" gate="1" x="373.38" y="109.22"/>
 <instance part="U2" gate="G$1" x="314.96" y="116.84" rot="MR0"/>
+<instance part="U$1" gate="G$1" x="177.8" y="2.54"/>
 </instances>
 <busses>
